File: Hardware/CORS_Time_Reference.sch (EAGLE design)
At the start: 240 parts, among them J10 ANTENNA-SMA-GROUNDEDEDGE_SMA, J11 Vertical Qwiic Connector, J2 ANTENNA-SMA-GROUNDEDEDGE_SMA, J3 MICRO-SD-PUSH-PUSH-EXT-PIN, J4 Vertical Qwiic Connector, J7 ANTENNA-SMA-GROUNDEDEDGE_SMA, J9 MAGJACK-POE, U1 ESP-WROOM-32E, U10 POE_PSU-DP990X, U11 OPA344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

Commit message: v01 after proto review
Parts:
- added C16: 10uF, SparkFun-Capacitors:10UF-0805-25V-10%
- added C51, C52: 0.1uF, SparkFun-Capacitors:0.1UF-0603-25V-5%
- added C55: 10uF, SparkFun-Capacitors:10UF-0603-6.3V-20%
- added C56: 2.2uF, SparkFun-Capacitors:2.2UF-0603-10V-20%
- C20: value 2.2uF -> 10uF; device SparkFun-Capacitors:2.2UF-0603-10V-20% -> SparkFun-Capacitors:10UF-0603-6.3V-20%
Connections:
- net N$44 renamed MEAS
- net 3.3V_SW: now also C52.1, C55.1, C56.1
- net 5V: now also C16.1, C51.1
- net GND: now also C16.2, C51.2, C52.2, C55.2, C56.2
Other:
- note added: "v01"
- note removed: "v10"
- moved on the sheet: D8, J13, J5, R27, R28, SHLD3

Commit message: Add CONN-17279
Parts:
- J13: device Terminal_Connectors:CONN_10 -> SparkFun-Connectors:CONN_10_3.5MM_RA_HEADER
Changed lines of the file:
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@@
 <part name="VUSB2" library="SparkFun-Connectors" deviceset="TEST-POINT" device="POGO_PTH" value="TEST-POINTPOGO_PTH"/>
 <part name="VUSB" library="SparkFun-Connectors" deviceset="TEST-POINT" device="POGO_PTH" value="TEST-POINTPOGO_PTH"/>
-<part name="J13" library="Terminal_Connectors" deviceset="CONN_10" device=""/>
 <part name="ANT_DET" library="SparkFun-Connectors" deviceset="TEST-POINT" device="POGO_PTH" value="TEST-POINTPOGO_PTH"/>
 <part name="ANT_SHT" library="SparkFun-Connectors" deviceset="TEST-POINT" device="POGO_PTH" value="TEST-POINTPOGO_PTH"/>
@@
 <part name="C56" library="SparkFun-Capacitors" deviceset="2.2UF" device="-0603-10V-20%" value="2.2uF"/>
 <part name="GND73" library="SparkFun-PowerSymbols" deviceset="GND" device=""/>
+<part name="J13" library="SparkFun-Connectors" deviceset="CONN_10" device="_3.5MM_RA_HEADER"/>
 </parts>
 <sheets>
@@
 <instance part="VUSB2" gate="G$1" x="25.4" y="35.56" smashed="yes" rot="R90"/>
 <instance part="VUSB" gate="G$1" x="119.38" y="208.28" smashed="yes"/>
-<instance part="J13" gate="JP1" x="152.4" y="20.32" smashed="yes">
-<attribute name="VALUE" x="149.86" y="5.334" size="1.778" layer="96" font="vector"/>
-<attribute name="NAME" x="149.86" y="36.068" size="1.778" layer="95" font="vector"/>
-</instance>
 <instance part="ANT_DET" gate="G$1" x="317.5" y="215.9" smashed="yes" rot="R90"/>
 <instance part="ANT_SHT" gate="G$1" x="312.42" y="193.04" smashed="yes" rot="R90"/>
@@
 <attribute name="VALUE" x="325.12" y="86.106" size="1.778" layer="96" align="top-center"/>
 </instance>
+<instance part="J13" gate="J1" x="149.86" y="27.94" smashed="yes">
+<attribute name="VALUE" x="149.86" y="5.334" size="1.778" layer="96" font="vector"/>
+<attribute name="NAME" x="149.86" y="36.068" size="1.778" layer="95" font="vector"/>
+</instance>
 </instances>
 <busses>
@@
 </segment>
 <segment>
-<pinref part="J13" gate="JP1" pin="9"/>
 <wire x1="160.02" y1="30.48" x2="162.56" y2="30.48" width="0.1524" layer="91"/>
 <pinref part="GND81" gate="1" pin="GND"/>
 <wire x1="162.56" y1="7.62" x2="162.56" y2="30.48" width="0.1524" layer="91"/>
+<pinref part="J13" gate="J1" pin="9"/>
 </segment>
 <segment>
@@
 </segment>
 <segment>
-<pinref part="J13" gate="JP1" pin="8"/>
 <wire x1="160.02" y1="27.94" x2="170.18" y2="27.94" width="0.1524" layer="91"/>
 <pinref part="SUPPLY51" gate="G$1" pin="3.3V_SW"/>
 <wire x1="170.18" y1="27.94" x2="170.18" y2="35.56" width="0.1524" layer="91"/>
+<pinref part="J13" gate="J1" pin="8"/>
 </segment>
 <segment>
@@
 <segment>
 <label x="170.18" y="25.4" size="1.27" layer="95" xref="yes"/>
-<pinref part="J13" gate="JP1" pin="7"/>
 <wire x1="160.02" y1="25.4" x2="170.18" y2="25.4" width="0.1524" layer="91"/>
+<pinref part="J13" gate="J1" pin="7"/>
 </segment>
 </net>
@@
 <segment>
 <label x="170.18" y="22.86" size="1.27" layer="95" xref="yes"/>
-<pinref part="J13" gate="JP1" pin="6"/>
 <wire x1="160.02" y1="22.86" x2="170.18" y2="22.86" width="0.1524" layer="91"/>
+<pinref part="J13" gate="J1" pin="6"/>
 </segment>
 </net>
@@
 </segment>
 <segment>
-<pinref part="J13" gate="JP1" pin="10"/>
 <wire x1="160.02" y1="33.02" x2="162.56" y2="33.02" width="0.1524" layer="91"/>
 <pinref part="SUPPLY53" gate="G$1" pin="5V"/>
 <wire x1="162.56" y1="33.02" x2="162.56" y2="35.56" width="0.1524" layer="91"/>
+<pinref part="J13" gate="J1" pin="10"/>
 </segment>
 <segment>
@@
 <segment>
 <label x="170.18" y="10.16" size="1.27" layer="95" xref="yes"/>
-<pinref part="J13" gate="JP1" pin="1"/>
 <wire x1="160.02" y1="10.16" x2="170.18" y2="10.16" width="0.1524" layer="91"/>
+<pinref part="J13" gate="J1" pin="1"/>
 </segment>
 </net>
@@
 <segment>
 <label x="170.18" y="15.24" size="1.27" layer="95" xref="yes"/>
-<pinref part="J13" gate="JP1" pin="3"/>
 <wire x1="160.02" y1="15.24" x2="165.1" y2="15.24" width="0.1524" layer="91"/>
 <pinref part="RXD" gate="G$1" pin="1"/>
@@
 <wire x1="165.1" y1="30.48" x2="165.1" y2="15.24" width="0.1524" layer="91"/>
 <junction x="165.1" y="15.24"/>
+<pinref part="J13" gate="J1" pin="3"/>
 </segment>
 </net>
@@
 <segment>
 <label x="170.18" y="12.7" size="1.27" layer="95" xref="yes"/>
-<pinref part="J13" gate="JP1" pin="2"/>
 <wire x1="160.02" y1="12.7" x2="167.64" y2="12.7" width="0.1524" layer="91"/>
 <pinref part="TXD" gate="G$1" pin="1"/>
@@
 <wire x1="167.64" y1="30.48" x2="167.64" y2="12.7" width="0.1524" layer="91"/>
 <junction x="167.64" y="12.7"/>
+<pinref part="J13" gate="J1" pin="2"/>
 </segment>
 </net>
@@
 </segment>
 <segment>
-<pinref part="J13" gate="JP1" pin="4"/>
 <wire x1="160.02" y1="17.78" x2="170.18" y2="17.78" width="0.1524" layer="91"/>
 <label x="170.18" y="17.78" size="1.27" layer="95" xref="yes"/>
+<pinref part="J13" gate="J1" pin="4"/>
 </segment>
 </net>
@@
 </segment>
 <segment>
-<pinref part="J13" gate="JP1" pin="5"/>
 <wire x1="160.02" y1="20.32" x2="170.18" y2="20.32" width="0.1524" layer="91"/>
 <label x="170.18" y="20.32" size="1.27" layer="95" xref="yes"/>
+<pinref part="J13" gate="J1" pin="5"/>
 </segment>
 </net>

Commit message: Change ESP32 SMA to RP
Parts:
- J7: value ANTENNA-SMA-GROUNDEDEDGE_SMA -> ANTENNA-SMA-GROUNDEDEDGE_RPSMA; device SparkFun-RF:ANTENNA-SMA-GROUNDEDEDGE_SMA -> SparkFun-RF:ANTENNA-SMA-GROUNDEDEDGE_RPSMA
Changed lines of the file:
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@@
 <part name="SUPPLY32" library="SparkFun-PowerSymbols" deviceset="5V" device=""/>
 <part name="GND57" library="SparkFun-PowerSymbols" deviceset="GND" device=""/>
-<part name="J7" library="SparkFun-RF" deviceset="ANTENNA-SMA-GROUNDED" device="EDGE_SMA"/>
+<part name="J7" library="SparkFun-RF" deviceset="ANTENNA-SMA-GROUNDED" device="EDGE_RPSMA" value="ANTENNA-SMA-GROUNDEDEDGE_RPSMA"/>
 <part name="J8" library="SparkFun-Connectors" deviceset="U.FL2PIN" device="-REDUCED-FOOTPRINT"/>
 <part name="GND59" library="SparkFun-PowerSymbols" deviceset="GND" device=""/>
