File: Hardware/Production/CORS_Time_Reference-Panel.brd (EAGLE design)
At the start: 166.1 x 131.1 mm, 393 parts, among them J10 ANTENNA-SMA-GROUNDEDEDGE_SMA, J11 Vertical Qwiic Connector, J2 ANTENNA-SMA-GROUNDEDEDGE_SMA, J3 MICRO-SD-PUSH-PUSH-EXT-PIN, J4 Vertical Qwiic Connector, J7 ANTENNA-SMA-GROUNDEDEDGE_SMA, J9 MAGJACK-POE, U1 ESP-WROOM-32E, U10 POE_PSU-DP990X, U11 OPA344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

Commit message: v01 after proto review
Parts:
- removed LOGO9: OSHW-LOGOS, SparkFun-Aesthetics:OSHW-LOGO-S
- added C16: 10uF, SparkFun-Capacitors:0805
- added C51, C52: 0.1uF, SparkFun-Capacitors:0603
- added C55: 10uF, SparkFun-Capacitors:0603
- added C56: 2.2uF, SparkFun-Capacitors:0603
- added U$152, U$153: (no value), output:RTK5#SVG0
- C20: value 2.2uF -> 10uF
- moved LOGO4 73.3 mm to (58.4, 3.81)
- moved U$84 2.03 mm to (41.0, 45.0)
Connections:
- net N$44 renamed MEAS
- net 3.3V_SW: now also C52.1, C55.1, C56.1
- net 5V: now also C16.1, C51.1
- net GND: now also C16.2, C51.2, C52.2, C55.2, C56.2
Routing:
- net 3.3V_SW: track 331.7 -> 348.0 mm, vias 15 -> 16
- net MEAS: track 14.0 -> 0.76 mm, vias 0 -> 10
- net 5V: track 215.7 -> 225.2 mm
- net GND: vias 321 -> 326
- added copper zone on layer 1, net MEAS
- added copper zone on layer 15, net MEAS
- added copper zone on layer 16, net MEAS
Other:
- board text added: "v01"
- board text removed: "v10"

Commit message: Add CONN-17279
Parts:
- J13: device Terminal_Connectors:1X10_SCREW_TERMINAL_3.5MM -> SparkFun-Connectors:1X10_SCREW_TERMINAL_3.5MM
Changed lines of the file:
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@@
 <element name="VUSB2" library="SparkFun-Connectors" package="1X01_NO_SILK" value="TEST-POINTPOGO_PTH" x="40.64" y="36.83" smashed="yes"/>
 <element name="VUSB" library="SparkFun-Connectors" package="1X01_NO_SILK" value="TEST-POINTPOGO_PTH" x="38.1" y="36.83" smashed="yes"/>
-<element name="J13" library="Terminal_Connectors" package="1X10_SCREW_TERMINAL_3.5MM" value="" x="67.31" y="97.79" smashed="yes" rot="R180">
+<element name="J13" library="SparkFun-Connectors" package="1X10_SCREW_TERMINAL_3.5MM" value="" x="67.31" y="97.79" smashed="yes" rot="R180">
 <attribute name="NAME" x="67.31" y="92.71" size="1.27" layer="25" rot="R180" align="bottom-center"/>
-<attribute name="PROD_ID" value="" x="67.31" y="97.79" size="1.778" layer="27" ratio="15" rot="R180" display="off"/>
+<attribute name="PROD_ID" value="CONN-17279" x="67.31" y="97.79" size="1.778" layer="27" ratio="15" rot="R180" display="off"/>
+<attribute name="STOREFRONT" value="PRT-21328" x="67.31" y="97.79" size="1.778" layer="27" ratio="15" rot="R180" display="off"/>
 <attribute name="VALUE" x="67.31" y="104.14" size="1.27" layer="27" rot="R180" align="bottom-center"/>
 </element>

Commit message: Change ESP32 SMA to RP
Parts:
- J7: value ANTENNA-SMA-GROUNDEDEDGE_SMA -> ANTENNA-SMA-GROUNDEDEDGE_RPSMA; device SparkFun-RF:SMA-EDGE -> SparkFun-RF:RP-SMA-EDGE
Changed lines of the file:
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@@
 <attribute name="NAME" x="138.557" y="3.175" size="0.6096" layer="26" font="vector" ratio="20" rot="MR270" align="bottom-center"/>
 </element>
-<element name="J7" library="SparkFun-RF" package="SMA-EDGE" value="ANTENNA-SMA-GROUNDEDEDGE_SMA" x="95.25" y="99.314" smashed="yes">
-<attribute name="PROD_ID" value="CONN-08289" x="86.36" y="113.284" size="1.778" layer="27" ratio="15" display="off"/>
+<element name="J7" library="SparkFun-RF" package="RP-SMA-EDGE" value="ANTENNA-SMA-GROUNDEDEDGE_RPSMA" x="95.25" y="99.314" smashed="yes">
+<attribute name="PROD_ID" value="CONN-00827" x="86.36" y="113.284" size="1.778" layer="27" ratio="15" display="off"/>
 </element>
 <element name="J8" library="SparkFun-Connectors" package="U.FL_REDUCED_FOOTPRINT" value="" x="95.25" y="88.9" smashed="yes" rot="R90">
