File: Front_Panel/CORS_Front_Panel.sch (EAGLE design)
At the start: 10 parts

Commit message: Update panels
Other:
- note added: "v02"
- note removed: "v01"
Changed lines of the file:
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@@
 <sheet>
 <plain>
-<text x="241.3" y="7.62" size="2.54" layer="94" font="vector">v01</text>
+<text x="241.3" y="7.62" size="2.54" layer="94" font="vector">v02</text>
 <text x="167.64" y="10.16" size="2.54" layer="94" font="vector">Paul Clark</text>
 </plain>
