File: Rear_Panel_Sticker/CORS_Rear_Panel.sch (EAGLE design)
At the start: 8 parts

Commit message: Update stickers
Parts:
- removed LOGO1: SFE_LOGO_NAME_FLAME.2_INCH, SparkFun-Aesthetics:SFE_LOGO_NAME_FLAME.2_INCH
Changed lines of the file:
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@@
 <part name="GND1" library="SparkFun-PowerSymbols" deviceset="GND" device=""/>
 <part name="ESP32_USB" library="CORS_Panels" deviceset="USB-C" device=""/>
-<part name="LOGO1" library="SparkFun-Aesthetics" deviceset="SFE_LOGO_NAME_FLAME" device=".2_INCH" value="SFE_LOGO_NAME_FLAME.2_INCH"/>
 <part name="U$13" library="CORS_Panels" deviceset="SMA" device=""/>
 <part name="U$14" library="CORS_Panels" deviceset="SMA" device=""/>
@@
 </instance>
 <instance part="ESP32_USB" gate="G$1" x="162.5" y="95" smashed="yes"/>
-<instance part="LOGO1" gate="G$1" x="85" y="2.5" smashed="yes"/>
 <instance part="U$13" gate="G$1" x="60.96" y="96.52" smashed="yes"/>
 <instance part="U$14" gate="G$1" x="78.74" y="96.52" smashed="yes"/>
